Commit message: update

File: urdf/ia_robot.urdf (robot description, URDF)
Before this commit: robot ia_robot, 19 links, 18 joints
Links:
- link LeftARM02: mass 2.5 -> 0.27589; geometry collision mesh filename=package://ia_robot/meshes/LeftARM02.STL; visual mesh filename=package://ia_robot/meshes/LeftARM02.STL
- link LeftARM03: mass 2 -> 0.47985; geometry collision mesh filename=package://ia_robot/meshes/LeftARM03.STL; visual mesh filename=package://ia_robot/meshes/LeftARM03.STL
- link LeftARM1: mass 1.822 -> 1.82195171111395; geometry collision mesh filename=package://ia_robot/meshes/LeftARM1.STL; visual mesh filename=package://ia_robot/meshes/LeftARM1.STL
- link LeftEnd: geometry collision mesh filename=package://ia_robot/meshes/LeftEnd.STL; visual mesh filename=package://ia_robot/meshes/LeftEnd.STL
- link LeftFrontWheelOrient1: mass 0.21206 -> 0.212057188740176; geometry collision mesh filename=package://ia_robot/meshes/LeftFrontWheelOrient1.STL; visual mesh filename=package://ia_robot/meshes/LeftFrontWheelOrient1.STL
- link LeftFrontWheelOrient2: mass 1 -> 0.427167332080997; geometry collision mesh filename=package://ia_robot/meshes/LeftFrontWheelOrient2.STL; visual mesh filename=package://ia_robot/meshes/LeftFrontWheelOrient2.STL
- link LeftFrontwheel: mass 5 -> 3.61818023273865; geometry collision mesh filename=package://ia_robot/meshes/LeftFrontwheel.STL; visual mesh filename=package://ia_robot/meshes/LeftFrontwheel.STL
- link RightARM1: geometry collision mesh filename=package://ia_robot/meshes/RightARM1.STL; visual mesh filename=package://ia_robot/meshes/RightARM1.STL
- link RightARM3: mass 2 -> 0.47985; geometry collision mesh filename=package://ia_robot/meshes/RightARM3.STL; visual mesh filename=package://ia_robot/meshes/RightARM3.STL
- link RightEnd: geometry collision mesh filename=package://ia_robot/meshes/RightEnd.STL; visual mesh filename=package://ia_robot/meshes/RightEnd.STL
- link RightFrontWheelOrient01: mass 0.21206 -> 0.212057174883898; geometry collision mesh filename=package://ia_robot/meshes/RightFrontWheelOrient01.STL; visual mesh filename=package://ia_robot/meshes/RightFrontWheelOrient01.STL
- link RightFrontWheelOrient1: mass 5 -> 3.61818023273865; geometry collision mesh filename=package://ia_robot/meshes/RightFrontWheelOrient1.STL; visual mesh filename=package://ia_robot/meshes/RightFrontWheelOrient1.STL
- link RightFrontWheelOrient2: mass 1 -> 0.427167332080998; geometry collision mesh filename=package://ia_robot/meshes/RightFrontWheelOrient2.STL; visual mesh filename=package://ia_robot/meshes/RightFrontWheelOrient2.STL
- link Rightbackorient: geometry collision mesh filename=package://ia_robot/meshes/Rightbackorient.STL; visual mesh filename=package://ia_robot/meshes/Rightbackorient.STL
- link Rightbackwheel: mass 5 -> 3.61818023273865; geometry collision mesh filename=package://ia_robot/meshes/Rightbackwheel.STL; visual mesh filename=package://ia_robot/meshes/Rightbackwheel.STL
- link RihgtARM2: mass 2.5 -> 0.27589; geometry collision mesh filename=package://ia_robot/meshes/RihgtARM2.STL; visual mesh filename=package://ia_robot/meshes/RihgtARM2.STL
- link base_link: mass 40.824 -> 42.189; geometry collision mesh filename=package://ia_robot/meshes/base_link.STL; visual mesh filename=package://ia_robot/meshes/base_link.STL
- link leftbackorient: geometry collision mesh filename=package://ia_robot/meshes/leftbackorient.STL; visual mesh filename=package://ia_robot/meshes/leftbackorient.STL
- link leftbackwheel: mass 5 -> 3.6182; geometry collision mesh filename=package://ia_robot/meshes/leftbackwheel.STL; visual mesh filename=package://ia_robot/meshes/leftbackwheel.STL
Joints:
- removed joint RightFrontWheelOrient1-1
- added joint RightFrontWheel: type continuous, parent RightFrontWheelOrient01, child RightFrontWheelOrient1, origin xyz=-0.00010607 0.0019972 -0.11 rpy=1.5708 0 0.053062, axis 0 0 -1, limit effort=50 velocity=0
- joint LeftARMJoint02: origin xyz=0.11738 0.046728 0.073 rpy=2.7627 -1.5708 0 -> xyz=0.12634 -0.0001172 0.073 rpy=3.1407 -1.5708 3.1416
- joint LeftARMJoint03: origin xyz=0.059196 -0.00067202 0.28311 rpy=-1.5708 1.192 -1.5822 -> xyz=0.059067 -0.003961 0.28311 rpy=1.5708 1.5699 1.5038; type revolute -> continuous
- joint LeftEndJoint: origin xyz=-0.65936 0.10584 -0.049114 rpy=-1.7017 -0.014293 -0.076285 -> xyz=-0.66222 0.086205 -0.049114 rpy=-1.7017 -0.0062132 -0.047629; type revolute -> continuous
- joint LeftFrontWheelOrient1-1: origin xyz=-0.17991 0.0058386 -0.0146 rpy=0 0 0 -> xyz=-0.179905283136192 0.00583858713100255 -0.0146000000000007 rpy=0 0 0
- joint LeftFrontwheel-1: origin xyz=-5.5247E-05 0.0019992 -0.11 rpy=1.5708 0 0.027627 -> xyz=-5.52466221374059E-05 0.00199923680706893 -0.11 rpy=1.5707963267949 0 0.0276268252558954
- joint RightARMJoint3: origin xyz=0.002656 0.05914 0.28311 rpy=1.5708 1.1923 -0.04493 -> xyz=0.058694 -0.0077252 0.28311 rpy=-1.5708 1.5707 1.4399; type revolute -> continuous
- joint RightEndJOINT: origin xyz=-0.65977 -0.10327 0.049114 rpy=1.4399 0.026 0.070847 -> xyz=-0.66559 -0.054292 0.049114 rpy=1.4399 0.00095434 0.00026273; type revolute -> continuous
- joint Rightbackwheel-1: axis -0.080582 0 -0.99675 -> -0.08058173506303 0 -0.996748004248933; origin xyz=-0.00016116 0.0019935 -0.11 rpy=1.5708 0 0 -> xyz=-0.000161163470126346 0.00199349600849796 -0.11 rpy=1.5707963267949 0 0
- joint RihgtARMJoint2: origin xyz=0.11738 -0.046728 0.073 rpy=-1.5708 0 1.1919 -> xyz=0.126339132538937 0.000117203456298176 0.0729999999999077 rpy=1.5707963267949 0 -1.56986863780086
