Commit message: update latest urdf

File: install/ia_robot/share/ia_robot/urdf/ia_robot.urdf (robot description, URDF)
Before this commit: robot ia_robot, 19 links, 18 joints
Links:
- link LeftARM02: geometry collision mesh filename=package://ia_robot/meshes/LeftARM02.stl; visual mesh filename=package://ia_robot/meshes/LeftARM02.stl
- link LeftARM03: geometry collision mesh filename=package://ia_robot/meshes/LeftARM03.stl; visual mesh filename=package://ia_robot/meshes/LeftARM03.stl
- link LeftARM1: geometry collision mesh filename=package://ia_robot/meshes/LeftARM1.stl; visual mesh filename=package://ia_robot/meshes/LeftARM1.stl
- link LeftEnd: geometry collision mesh filename=package://ia_robot/meshes/LeftEnd.stl; visual mesh filename=package://ia_robot/meshes/LeftEnd.stl
- link LeftFrontWheelOrient1: geometry collision mesh filename=package://ia_robot/meshes/LeftFrontWheelOrient1.stl; visual mesh filename=package://ia_robot/meshes/LeftFrontWheelOrient1.stl
- link LeftFrontWheelOrient2: geometry collision mesh filename=package://ia_robot/meshes/LeftFrontWheelOrient2.stl; visual mesh filename=package://ia_robot/meshes/LeftFrontWheelOrient2.stl
- link LeftFrontwheel: geometry collision mesh filename=package://ia_robot/meshes/LeftFrontwheel.stl; visual mesh filename=package://ia_robot/meshes/LeftFrontwheel.stl
- link RightARM1: geometry collision mesh filename=package://ia_robot/meshes/RightARM1.stl; visual mesh filename=package://ia_robot/meshes/RightARM1.stl
- link RightARM3: geometry collision mesh filename=package://ia_robot/meshes/RightARM3.stl; visual mesh filename=package://ia_robot/meshes/RightARM3.stl
- link RightEnd: geometry collision mesh filename=package://ia_robot/meshes/RightEnd.stl; visual mesh filename=package://ia_robot/meshes/RightEnd.stl
- link RightFrontWheelOrient01: geometry collision mesh filename=package://ia_robot/meshes/RightFrontWheelOrient01.stl; visual mesh filename=package://ia_robot/meshes/RightFrontWheelOrient01.stl
- link RightFrontWheelOrient1: geometry collision mesh filename=package://ia_robot/meshes/RightFrontWheelOrient1.stl; visual mesh filename=package://ia_robot/meshes/RightFrontWheelOrient1.stl
- link RightFrontWheelOrient2: geometry collision mesh filename=package://ia_robot/meshes/RightFrontWheelOrient2.stl; visual mesh filename=package://ia_robot/meshes/RightFrontWheelOrient2.stl
- link Rightbackorient: geometry collision mesh filename=package://ia_robot/meshes/Rightbackorient.stl; visual mesh filename=package://ia_robot/meshes/Rightbackorient.stl
- link Rightbackwheel: geometry collision mesh filename=package://ia_robot/meshes/Rightbackwheel.stl; visual mesh filename=package://ia_robot/meshes/Rightbackwheel.stl
- link RihgtARM2: geometry collision mesh filename=package://ia_robot/meshes/RihgtARM2.stl; visual mesh filename=package://ia_robot/meshes/RihgtARM2.stl
- link base_link: geometry collision mesh filename=package://ia_robot/meshes/base_link.stl; visual mesh filename=package://ia_robot/meshes/base_link.stl
- link leftbackorient: geometry collision mesh filename=package://ia_robot/meshes/leftbackorient.stl; visual mesh filename=package://ia_robot/meshes/leftbackorient.stl
- link leftbackwheel: geometry collision mesh filename=package://ia_robot/meshes/leftbackwheel.stl; visual mesh filename=package://ia_robot/meshes/leftbackwheel.stl

File: urdf/ia_robot.urdf (robot description, URDF)
Before this commit: robot ia_robot, 19 links, 18 joints
Links:
- link LeftARM02: geometry collision mesh filename=package://ia_robot/meshes/LeftARM02.stl; visual mesh filename=package://ia_robot/meshes/LeftARM02.stl
- link LeftARM03: geometry collision mesh filename=package://ia_robot/meshes/LeftARM03.stl; visual mesh filename=package://ia_robot/meshes/LeftARM03.stl
- link LeftARM1: geometry collision mesh filename=package://ia_robot/meshes/LeftARM1.stl; visual mesh filename=package://ia_robot/meshes/LeftARM1.stl
- link LeftEnd: geometry collision mesh filename=package://ia_robot/meshes/LeftEnd.stl; visual mesh filename=package://ia_robot/meshes/LeftEnd.stl
- link LeftFrontWheelOrient1: geometry collision mesh filename=package://ia_robot/meshes/LeftFrontWheelOrient1.stl; visual mesh filename=package://ia_robot/meshes/LeftFrontWheelOrient1.stl
- link LeftFrontWheelOrient2: geometry collision mesh filename=package://ia_robot/meshes/LeftFrontWheelOrient2.stl; visual mesh filename=package://ia_robot/meshes/LeftFrontWheelOrient2.stl
- link LeftFrontwheel: geometry collision mesh filename=package://ia_robot/meshes/LeftFrontwheel.stl; visual mesh filename=package://ia_robot/meshes/LeftFrontwheel.stl
- link RightARM1: geometry collision mesh filename=package://ia_robot/meshes/RightARM1.stl; visual mesh filename=package://ia_robot/meshes/RightARM1.stl
- link RightARM3: geometry collision mesh filename=package://ia_robot/meshes/RightARM3.stl; visual mesh filename=package://ia_robot/meshes/RightARM3.stl
- link RightEnd: geometry collision mesh filename=package://ia_robot/meshes/RightEnd.stl; visual mesh filename=package://ia_robot/meshes/RightEnd.stl
- link RightFrontWheelOrient01: geometry collision mesh filename=package://ia_robot/meshes/RightFrontWheelOrient01.stl; visual mesh filename=package://ia_robot/meshes/RightFrontWheelOrient01.stl
- link RightFrontWheelOrient1: geometry collision mesh filename=package://ia_robot/meshes/RightFrontWheelOrient1.stl; visual mesh filename=package://ia_robot/meshes/RightFrontWheelOrient1.stl
- link RightFrontWheelOrient2: geometry collision mesh filename=package://ia_robot/meshes/RightFrontWheelOrient2.stl; visual mesh filename=package://ia_robot/meshes/RightFrontWheelOrient2.stl
- link Rightbackorient: geometry collision mesh filename=package://ia_robot/meshes/Rightbackorient.stl; visual mesh filename=package://ia_robot/meshes/Rightbackorient.stl
- link Rightbackwheel: geometry collision mesh filename=package://ia_robot/meshes/Rightbackwheel.stl; visual mesh filename=package://ia_robot/meshes/Rightbackwheel.stl
- link RihgtARM2: geometry collision mesh filename=package://ia_robot/meshes/RihgtARM2.stl; visual mesh filename=package://ia_robot/meshes/RihgtARM2.stl
- link base_link: geometry collision mesh filename=package://ia_robot/meshes/base_link.stl; visual mesh filename=package://ia_robot/meshes/base_link.stl
- link leftbackorient: geometry collision mesh filename=package://ia_robot/meshes/leftbackorient.stl; visual mesh filename=package://ia_robot/meshes/leftbackorient.stl
- link leftbackwheel: geometry collision mesh filename=package://ia_robot/meshes/leftbackwheel.stl; visual mesh filename=package://ia_robot/meshes/leftbackwheel.stl
Joints:
- joint RihgtARMJoint2: origin xyz=0.126339132538937 0.000117203456298176 0.0729999999999077 rpy=1.5708 -1.5708 -1.5708 -> xyz=0.126339132538937 0.000117203456298176 0.0729999999999077 rpy=1.5708 1.5708 -1.5708
